File: _saved_ESP_multi_board.sch (KiCad schematic (older format))
At the start: 21 parts, among them P101 CONN_01X02, P102 CONN_01X06, P103 CONN_01X02, P104 CONN_01X06, P105 CONN_01X12, P106 CONN_01X03, P107 CONN_I2C_MPU6050, P108 CONN_PINES_DIG, SW101 SW_PUSH_SMALL, SW102 SPST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

Commit message: vesion simplificada, sin jumper y sinconectar los pines de int
Parts:
- removed SW102: SPST, Buttons_Switches_SMD:SW_SPST_REED_CT10-XXXX-G1, symbol SPST
- added SW102: SWITCH_INV, Buttons_Switches_ThroughHole:SW_Micro_SPST, symbol SWITCH_INV
Connections:
- net VCC: now also SW102.2
- net reg5to3_3V/VCC: now also SW102.1
Changed lines of the file:
@@
 LIBS:contrib
 LIBS:valves
-LIBS:figaro
-LIBS:ADC128D818
-LIBS:sensors-cache
+LIBS:ESP8266
+LIBS:stepper drivers
+LIBS:mpu-6050
+LIBS:MCP23008
+LIBS:microchip_adcdac
+LIBS:ESP_multi_board-cache
 EELAYER 25 0
 EELAYER END
@@
 L VCC #PWR06
 U 1 1 57125BE7
-P 850 1150
-F 0 "#PWR06" H 850 1000 50  0001 C CNN
-F 1 "VCC" H 850 1300 50  0000 C CNN
-F 2 "" H 850 1150 50  0000 C CNN
-F 3 "" H 850 1150 50  0000 C CNN
-	1    850  1150
+P 700 1250
+F 0 "#PWR06" H 700 1100 50  0001 C CNN
+F 1 "VCC" H 700 1400 50  0000 C CNN
+F 2 "" H 700 1250 50  0000 C CNN
+F 3 "" H 700 1250 50  0000 C CNN
+	1    700  1250
 	0    -1   -1   0
 $EndComp
@@
 NoConn ~ 7750 2050
 $Comp
-L SPST SW102
-U 1 1 57214B62
-P 1350 1150
-F 0 "SW102" H 1350 1250 50  0000 C CNN
-F 1 "SPST" H 1350 1050 50  0000 C CNN
-F 2 "Buttons_Switches_SMD:SW_SPST_REED_CT10-XXXX-G1" H 1350 1150 50  0001 C CNN
-F 3 "" H 1350 1150 50  0000 C CNN
-	1    1350 1150
-	1    0    0    -1
-$EndComp
+L SWITCH_INV SW102
+U 1 1 57214298
+P 1200 1250
+F 0 "SW102" H 1000 1400 50  0000 C CNN
+F 1 "SWITCH_INV" H 1050 1100 50  0000 C CNN
+F 2 "Buttons_Switches_ThroughHole:SW_Micro_SPST" H 1200 1250 50  0001 C CNN
+F 3 "" H 1200 1250 50  0000 C CNN
+	1    1200 1250
+	1    0    0    -1
+$EndComp
+Wire Wire Line
+	1850 1150 1700 1150
 $EndSCHEMATC
