File: _saved_ESP_multi_board.sch (KiCad schematic (older format))
At the start: 21 parts, among them P101 CONN_01X02, P102 CONN_01X06, P103 CONN_01X02, P104 CONN_01X06, P105 CONN_01X12, P106 CONN_01X03, P107 CONN_I2C_MPU6050, P108 CONN_PINES_DIG, SW101 SW_PUSH_SMALL, SW102 SWITCH_INV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

Commit message: routing
Parts:
- added D101: D, Diodes_ThroughHole:Diode_DO-35_SOD27_Horizontal_RM10, symbol D
- added IC101: L298, TO_SOT_Packages_THT:Multiwatt_15_Vertical, symbol L298
- added IC102: L293D, Housings_DIP:DIP-16_W7.62mm, symbol L293D
Connections:
- wire segments 82 -> 83
Other:
- moved on the sheet: P103, SW102
Changed lines of the file:
@@
 L CONN_01X02 P103
 U 1 1 57125BEB
-P 2050 2550
-F 0 "P103" H 2050 2700 50  0000 C CNN
-F 1 "CONN_01X02" V 2150 2550 50  0000 C CNN
-F 2 "Pin_Headers:Pin_Header_Angled_1x02" H 2050 2550 50  0001 C CNN
-F 3 "" H 2050 2550 50  0000 C CNN
-	1    2050 2550
+P 2400 2550
+F 0 "P103" H 2400 2700 50  0000 C CNN
+F 1 "CONN_01X02" V 2500 2550 50  0000 C CNN
+F 2 "Pin_Headers:Pin_Header_Angled_1x02" H 2400 2550 50  0001 C CNN
+F 3 "" H 2400 2550 50  0000 C CNN
+	1    2400 2550
 	0    -1   -1   0
 $EndComp
@@
 L PWR_FLAG #FLG018
 U 1 1 57154A7C
-P 2100 2750
-F 0 "#FLG018" H 2100 2845 50  0001 C CNN
-F 1 "PWR_FLAG" H 2100 2930 50  0000 C CNN
-F 2 "" H 2100 2750 50  0000 C CNN
-F 3 "" H 2100 2750 50  0000 C CNN
-	1    2100 2750
+P 2450 2750
+F 0 "#FLG018" H 2450 2845 50  0001 C CNN
+F 1 "PWR_FLAG" H 2450 2930 50  0000 C CNN
+F 2 "" H 2450 2750 50  0000 C CNN
+F 3 "" H 2450 2750 50  0000 C CNN
+	1    2450 2750
 	0    1    1    0
 $EndComp
@@
 L VCC #PWR019
 U 1 1 57154E13
-P 2100 2950
-F 0 "#PWR019" H 2100 2800 50  0001 C CNN
-F 1 "VCC" H 2100 3100 50  0000 C CNN
-F 2 "" H 2100 2950 50  0000 C CNN
-F 3 "" H 2100 2950 50  0000 C CNN
-	1    2100 2950
+P 2450 2950
+F 0 "#PWR019" H 2450 2800 50  0001 C CNN
+F 1 "VCC" H 2450 3100 50  0000 C CNN
+F 2 "" H 2450 2950 50  0000 C CNN
+F 3 "" H 2450 2950 50  0000 C CNN
+	1    2450 2950
 	-1   0    0    1
 $EndComp
@@
 L SWITCH_INV SW102
 U 1 1 57214298
-P 1500 2850
-F 0 "SW102" H 1300 3000 50  0000 C CNN
-F 1 "SWITCH_INV" H 1350 2700 50  0000 C CNN
-F 2 "Buttons_Switches_ThroughHole:SW_Micro_SPST" H 1500 2850 50  0001 C CNN
-F 3 "" H 1500 2850 50  0000 C CNN
-	1    1500 2850
+P 1850 2850
+F 0 "SW102" H 1650 3000 50  0000 C CNN
+F 1 "SWITCH_INV" H 1700 2700 50  0000 C CNN
+F 2 "Buttons_Switches_ThroughHole:SW_Micro_SPST" H 1850 2850 50  0001 C CNN
+F 3 "" H 1850 2850 50  0000 C CNN
+	1    1850 2850
 	1    0    0    -1
 $EndComp
@@
 Connection ~ 1250 4850
 Wire Wire Line
-	2100 2750 2100 2950
+	2450 2750 2450 2950
 Connection ~ 6750 1650
 Wire Wire Line
@@
 Wire Wire Line
 	4200 5850 4450 5850
+$Comp
+L D D101
+U 1 1 57231093
+P 1150 2850
+F 0 "D101" H 1150 2950 50  0000 C CNN
+F 1 "D" H 1150 2750 50  0000 C CNN
+F 2 "Diodes_ThroughHole:Diode_DO-35_SOD27_Horizontal_RM10" H 1150 2850 50  0001 C CNN
+F 3 "" H 1150 2850 50  0000 C CNN
+	1    1150 2850
+	1    0    0    -1
+$EndComp
+Wire Wire Line
+	1350 2850 1300 2850
+$Comp
+L L293D IC102
+U 1 1 5723ED74
+P 1950 6400
+F 0 "IC102" H 1550 7300 50  0000 L BNN
+F 1 "L293D" H 1550 5400 50  0000 L BNN
+F 2 "Housings_DIP:DIP-16_W7.62mm" H 1950 6550 50  0001 C CNN
+F 3 "" H 1950 6400 60  0000 C CNN
+	1    1950 6400
+	1    0    0    -1
+$EndComp
+$Comp
+L L298 IC101
+U 1 1 5723EDEF
+P 450 6200
+F 0 "IC101" H -32 6935 50  0000 L BNN
+F 1 "L298" H -9  5552 50  0000 L BNN
+F 2 "TO_SOT_Packages_THT:Multiwatt_15_Vertical" H 450 6350 50  0001 C CNN
+F 3 "" H 450 6200 60  0000 C CNN
+	1    450  6200
+	1    0    0    -1
+$EndComp
 $EndSCHEMATC
