File: reg5to3_3V.sch (KiCad schematic (older format))
At the start: 3 parts, among them U1 LD1117S33TR

Commit message: Actualizadas huellas de acuerdo a los componentes de Mouser
Parts:
- C2: footprint Capacitors_SMD:C_1206 -> Capacitors_SMD:C_0805_HandSoldering
Changed lines of the file:
@@
 F 0 "C2" H 4125 3150 50  0000 L CNN
 F 1 "100n" H 4125 2950 50  0000 L CNN
-F 2 "Capacitors_SMD:C_1206" H 4138 2900 50  0001 C CNN
+F 2 "Capacitors_SMD:C_0805_HandSoldering" H 4138 2900 50  0001 C CNN
 F 3 "" H 4100 3050 50  0000 C CNN
 	1    4100 3050
